File: Power.sch (KiCad schematic (older format))
At the start: 85 parts, among them J1 PhoneJack, J2 DB15, P3 I2C_EXT, P4 I2C_EXT, P5 UART_EXT, P6 I2C_EXT, P7 I2C_EXT, U1 LM358, U2 LM358, U3 LT8471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

Commit message: Work in progress
Parts:
- C6, C7: symbol CPSMALL -> CPsmall
- F1: symbol Fuse -> FUSE
- JP3, JP4: symbol Jumper -> JUMPER
Connections:
- wire segments 240 -> 238
Other:
- moved on the sheet: R12, R13, R14, R15, R16, R17, R22, R23, TP_GND1, TP_GND5, U7

Commit message: Work in progress
Parts:
- C10, C11, C14, C15, C16, C17: value 2.2uF -> 2.2u; footprint Capacitors_SMD:C_0603 -> Capacitors_Tantalum_SMD:TantalC_SizeD_EIA-7343_HandSoldering
- C12, C13, C9: value 0.01uF -> 10n; footprint Capacitors_SMD:C_0603 -> Capacitors_SMD:C_0805_HandSoldering
- C18, C19: value 47uF -> 47u; footprint Capacitors_SMD:C_0603 -> Capacitors_Tantalum_SMD:TantalC_SizeE_EIA-7360_HandSoldering
- C2, C3: value 1uF -> 1u; footprint Capacitors_SMD:C_0603 -> Capacitors_SMD:C_0805_HandSoldering
- C20, C21: value 10uF -> 10u; footprint Capacitors_SMD:C_0603 -> Capacitors_Tantalum_SMD:TantalC_SizeE_EIA-7360_HandSoldering
- C4, C5: value 1nF -> 1n; footprint Capacitors_SMD:C_0603 -> Capacitors_SMD:C_0805_HandSoldering
- C6, C7: footprint ~ -> Capacitors_Tantalum_SMD:TantalC_SizeE_EIA-7360_HandSoldering
- C8: value 0.01uf -> 10n; footprint Capacitors_SMD:C_0603 -> Capacitors_SMD:C_0805_HandSoldering
- D1, D2, D3, D4: footprint Diodes_SMD:D_SMC_Standard -> Diodes_SMD:SMC_Handsoldering
- J1: footprint Connectors:JACK_ALIM -> Connect:JACK_ALIM
- J2: footprint Connectors:DB15MC -> Connect:DB15MC
- JP3, JP4: footprint Wire_Connections_Bridges:WireConnection_2.00mmDrill -> Pin_Headers:Pin_Header_Angled_1x02
- L1, L2, L3, L4, L5, L6: footprint (none) -> Inductors:SELF-WE-TPC_M
- MR1, U5, U6, U7: footprint LEDs:LED_1206 -> Diodes_SMD:SMC_Handsoldering
- R10, R11, R12, R13, R14, R15, R16, R17, R19, R22, R23, R24, R25, R26, R27, R28, R4, R5, R6, R7, R8, R9: footprint Resistors_SMD:R_1206 -> Resistors_SMD:R_0805_HandSoldering
- R18: value 216K -> 220k; footprint Resistors_SMD:R_1206 -> Resistors_SMD:R_0805_HandSoldering
- R20, R21: value 215K -> 220k; footprint Resistors_SMD:R_1206 -> Resistors_SMD:R_0805_HandSoldering
- TP_-3V3_400mA1, TP_3V3_1.5A1, TP_3V3_400mA1, TP_5V_500mA1, TP_GND1, TP_GND2, TP_GND3, TP_GND4, TP_GND5, TP_VRout1, TP_Vadj1, TP_Vout1: footprint (none) -> Measurement_Points:Measurement_Point_Square-SMD-Pad_Big
- U1, U2: footprint Housings_DIP:DIP-8_W10.16mm -> SMD_Packages:SOIC-8-N
- U1: footprint (none) -> SMD_Packages:SOIC-8-N
- U3, U4: footprint Housings_DFN_QFN:QFN-28-1EP_4x5mm_Pitch0.5mm -> SMD_Packages:SSOP-20
