File: rp_hw.sch (KiCad schematic (older format))
At the start: 9 parts, among them IC1 AT24LC64-I/SN, P1 CONN_02X13, P2 CONN_02X13

Commit message: Work in progress
Parts:
- IC1: footprint Housings_SOIC:SOIC-8_3.9x4.9mm_Pitch1.27mm -> SMD_Packages:SOIC-8-N
Changed lines of the file:
@@
 $EndComp
 $Comp
-L GND #PWR5
+L GND #PWR01
 U 1 1 56DF8149
 P 8210 1910
-F 0 "#PWR5" H 8210 1660 50  0001 C CNN
+F 0 "#PWR01" H 8210 1660 50  0001 C CNN
 F 1 "GND" H 8210 1760 50  0000 C CNN
 F 2 "" H 8210 1910 50  0000 C CNN
@@
 CLKN
 $Comp
-L GND #PWR6
+L GND #PWR02
 U 1 1 56DF83FE
 P 8820 1985
-F 0 "#PWR6" H 8820 1735 50  0001 C CNN
+F 0 "#PWR02" H 8820 1735 50  0001 C CNN
 F 1 "GND" H 8820 1835 50  0000 C CNN
 F 2 "" H 8820 1985 50  0000 C CNN
@@
 NoConn ~ 9830 4640
 $Comp
-L GND #PWR7
+L GND #PWR03
 U 1 1 56DF8BFD
 P 9940 4850
-F 0 "#PWR7" H 9940 4600 50  0001 C CNN
+F 0 "#PWR03" H 9940 4600 50  0001 C CNN
 F 1 "GND" H 9940 4700 50  0000 C CNN
 F 2 "" H 9940 4850 50  0000 C CNN
@@
 F 0 "IC1" H 5665 1600 50  0000 C CNN
 F 1 "AT24LC64-I/SN" H 6165 1050 50  0000 C CNN
-F 2 "Housings_SOIC:SOIC-8_3.9x4.9mm_Pitch1.27mm" H 5865 1350 50  0000 C CIN
+F 2 "SMD_Packages:SOIC-8-N" H 5865 1350 50  0000 C CIN
 F 3 "" H 5865 1350 50  0000 C CNN
 	1    5865 1350
@@
 +3V3D
 $Comp
-L GND #PWR3
+L GND #PWR04
 U 1 1 56E4BB4A
 P 5245 1320
-F 0 "#PWR3" H 5245 1070 50  0001 C CNN
+F 0 "#PWR04" H 5245 1070 50  0001 C CNN
 F 1 "GND" H 5245 1170 50  0000 C CNN
 F 2 "" H 5245 1320 50  0000 C CNN
@@
 $EndComp
 $Comp
-L GND #PWR4
+L GND #PWR05
 U 1 1 56E4BBA4
 P 5865 1870
-F 0 "#PWR4" H 5865 1620 50  0001 C CNN
+F 0 "#PWR05" H 5865 1620 50  0001 C CNN
 F 1 "GND" H 5865 1720 50  0000 C CNN
 F 2 "" H 5865 1870 50  0000 C CNN
@@
 $EndComp
 $Comp
-L GND #PWR2
+L GND #PWR06
 U 1 1 56E4C2C9
 P 4960 2275
-F 0 "#PWR2" H 4960 2025 50  0001 C CNN
+F 0 "#PWR06" H 4960 2025 50  0001 C CNN
 F 1 "GND" H 4960 2125 50  0000 C CNN
 F 2 "" H 4960 2275 50  0000 C CNN
@@
 	4660 1450 4660 1615
 $Comp
-L GND #PWR1
+L GND #PWR07
 U 1 1 56E4CB70
 P 4660 1615
-F 0 "#PWR1" H 4660 1365 50  0001 C CNN
+F 0 "#PWR07" H 4660 1365 50  0001 C CNN
 F 1 "GND" H 4660 1465 50  0000 C CNN
 F 2 "" H 4660 1615 50  0000 C CNN
@@
 Connection ~ 10330 1935
 $Comp
-L GND #PWR8
+L GND #PWR08
 U 1 1 56E4E174
 P 10330 2005
-F 0 "#PWR8" H 10330 1755 50  0001 C CNN
+F 0 "#PWR08" H 10330 1755 50  0001 C CNN
 F 1 "GND" H 10330 1855 50  0000 C CNN
 F 2 "" H 10330 2005 50  0000 C CNN
@@
 	6810 850  6810 900
 Wire Wire Line
-	8210 1230 8210 1400
-Wire Wire Line
 	8210 1700 8210 1910
+Wire Wire Line
+	8210 1235 8210 1400
 $EndSCHEMATC
